Commit message: Fix new URDFs

File: urdf/cobot0.urdf.xacro (robot description, xacro)
@@ -1,7 +1,7 @@
 <?xml version="1.0" ?>
 <robot name="cobot0" xmlns:xacro="http://www.ros.org/wiki/xacro">
-    <xacro:include filename="$(find ar3_description)/urdf/create_ar3.xacro" />
+    <xacro:include filename="$(find ar3_description)/urdf/inc/create_ar3.xacro" />
     <link name="base_link"></link>
-    <xacro:ar3
+    <xacro:create_ar3
         prefix="cobot0"
         origin_xyz="0 0 0"

File: urdf/cobot1.urdf.xacro (robot description, xacro)
@@ -1,7 +1,7 @@
 <?xml version="1.0" ?>
-<robot name="cobot0" xmlns:xacro="http://www.ros.org/wiki/xacro">
-    <xacro:include filename="$(find ar3_description)/urdf/create_ar3.xacro" />
+<robot name="cobot1" xmlns:xacro="http://www.ros.org/wiki/xacro">
+    <xacro:include filename="$(find ar3_description)/urdf/inc/create_ar3.xacro" />
     <link name="base_link"></link>
-    <xacro:ar3
+    <xacro:create_ar3
         prefix="cobot1"
         origin_xyz="0 0 0"

File: urdf/inc/create_ar3.xacro (robot description, xacro)
@@ -18,5 +18,5 @@
     <!-- Base of AR3 -->
     <xacro:create_link
-      link_name = "{prefix}_base"
+      link_name = "${prefix}_base"
       mesh_package = "ar3_description"
       mesh_name = "base"
@@ -24,103 +24,103 @@
     <!-- Arm links -->
     <xacro:create_link
-      link_name = "{prefix}_link_0"
+      link_name = "${prefix}_link_0"
       mesh_package = "ar3_description"
       mesh_name = "link_0"
     />
     <xacro:create_link
-      link_name = "{prefix}_link_1"
+      link_name = "${prefix}_link_1"
       mesh_package = "ar3_description"
       mesh_name = "link_1"
     />
     <xacro:create_link
-      link_name = "{prefix}_link_2"
+      link_name = "${prefix}_link_2"
       mesh_package = "ar3_description"
       mesh_name = "link_2"
     />
     <xacro:create_link
-      link_name = "{prefix}_link_3"
+      link_name = "${prefix}_link_3"
       mesh_package = "ar3_description"
       mesh_name = "link_3"
     />
     <xacro:create_link
-      link_name = "{prefix}_link_4"
+      link_name = "${prefix}_link_4"
       mesh_package = "ar3_description"
       mesh_name = "link_4"
     />
     <xacro:create_link
-      link_name = "{prefix}_link_5"
+      link_name = "${prefix}_link_5"
       mesh_package = "ar3_description"
       mesh_name = "link_5"
     />
     <!-- Fixed joint between AR3 base and parent link -->
-    <joint name="{prefix}_base_joint" type="fixed">
-      <origin xyz="{origin_xyz}" rpy="{origin_rpy}" />
-      <parent link="{parent_link}" />
-      <child link="{prefix}_base" />
+    <joint name="${prefix}_base_joint" type="fixed">
+      <origin xyz="${origin_xyz}" rpy="${origin_rpy}" />
+      <parent link="${parent_link}" />
+      <child link="${prefix}_base" />
     </joint>
     <!-- Arm Joints -->
       <xacro:create_joint
-      name = "{prefix}_joint_0"
-      parent = "{prefix}_base"
-      child = "{prefix}_link_0"
+      name = "${prefix}_joint_0"
+      parent = "${prefix}_base"
+      child = "${prefix}_link_0"
       origin = "0 0 0.0872"
       axis = "0 0 1"
-      min = "-100"
-      max = "165"
+      min_deg = "-100"
+      max_deg = "165"
       velocity = "80"
       effort = "3.5"
     />
     <xacro:create_joint
-      name = "{prefix}_joint_1"
-      parent = "{prefix}_link_0"
-      child = "{prefix}_link_1"
+      name = "${prefix}_joint_1"
+      parent = "${prefix}_link_0"
+      child = "${prefix}_link_1"
       origin = "0.0642 0 0.0831"
       axis = "0 1 0"
-      min = "-55"
-      max = "43"
+      min_deg = "-55"
+      max_deg = "43"
       velocity = "60"
       effort = "20"
     />
     <xacro:create_joint
-      name = "{prefix}_joint_2"
-      parent = "{prefix}_link_1"
-      child = "{prefix}_link_2"
+      name = "${prefix}_joint_2"
+      parent = "${prefix}_link_1"
+      child = "${prefix}_link_2"
       origin = "0 0 0.3050"
       axis = "0 1 0"
-      min = "-160"
-      max = "125"
+      min_deg = "-160"
+      max_deg = "125"
       velocity = "160"
       effort = "10"
     />
     <xacro:create_joint
-      name = "{prefix}_joint_3"
-      parent = "{prefix}_link_2"
-      child = "{prefix}_link_3"
+      name = "${prefix}_joint_3"
+      parent = "${prefix}_link_2"
+      child = "${prefix}_link_3"
       origin = "0 0 0.0356"
       axis = "0 0 1"
-      min = "-160"
-      max = "135"
+      min_deg = "-160"
+      max_deg = "135"
       velocity = "240"
       effort = "3"
     />
     <xacro:create_joint
-      name = "{prefix}_joint_4"
-      parent = "{prefix}_link_3"
-      child = "{prefix}_link_4"
+      name = "${prefix}_joint_4"
+      parent = "${prefix}_link_3"
+      child = "${prefix}_link_4"
       origin = "0 0 0.1873"
       axis = "0 1 0"
-      min = "-98"
-      max = "98"
+      min_deg = "-98"
+      max_deg = "98"
       velocity = "200"
       effort = "0.1"
     />
     <xacro:create_joint
-      name = "{prefix}_joint_5"
-      parent = "{prefix}_link_4"
-      child = "{prefix}_link_5"
+      name = "${prefix}_joint_5"
+      parent = "${prefix}_link_4"
+      child = "${prefix}_link_5"
       origin = "0 0 0.0199"
       axis = "0 0 1"
-      min = "-150"
-      max = "140"
+      min_deg = "-150"
+      max_deg = "140"
       velocity = "1500"
       effort = "3"

File: urdf/inc/create_joint.xacro (robot description, xacro)
@@ -7,18 +7,18 @@
     origin
     axis
-    min
-    max
+    min_deg
+    max_deg
     velocity
     effort
   ">
-    <joint name="{name}" type="revolute">
-      <parent link="{parent}" />
-      <child link="{child}" />
+    <joint name="${name}" type="revolute">
+      <parent link="${parent}" />
+      <child link="${child}" />
       <origin xyz="${origin}" rpy="0 0 0" />
       <axis xyz="${axis}" />
       <limit
         effort="${effort}"
-        lower="${min*pi/180}"
-        upper="${max*pi/180}"
+        lower="${min_deg*pi/180}"
+        upper="${max_deg*pi/180}"
         velocity="${velocity*pi/180}"
       />

File: urdf/two_cobots.urdf.xacro (robot description, xacro)
@@ -1,7 +1,7 @@
 <?xml version="1.0" ?>
-<robot name="cobot0" xmlns:xacro="http://www.ros.org/wiki/xacro">
-    <xacro:include filename="$(find ar3_description)/urdf/create_ar3.xacro" />
+<robot name="two_cobots" xmlns:xacro="http://www.ros.org/wiki/xacro">
+    <xacro:include filename="$(find ar3_description)/urdf/inc/create_ar3.xacro" />
     <link name="base_link"></link>
-    <xacro:ar3
+    <xacro:create_ar3
         prefix="cobot0"
         origin_xyz="0 0 0"
@@ -9,8 +9,8 @@
         parent_link="base_link"
     />
-    <xacro:ar3
+    <xacro:create_ar3
         prefix="cobot1"
         origin_xyz="1.9 0 0"
-        origin_rpy="0 0 0"
+        origin_rpy="0 0 ${pi}"
         parent_link="base_link"
     />

Commit message: Cobot1

File: urdf/cobot0.urdf.xacro (robot description, xacro)
@@ -5,5 +5,5 @@
     <xacro:create_ar3
         prefix="cobot0"
-        origin_xyz="-0.39329375 0 0"
+        origin_xyz="-0.39129375 -0.018 0"
         origin_rpy="0 0 ${-pi/2}"
         parent_link="base_link"

File: urdf/inc/create_ar3.xacro (robot description, xacro)
@@ -99,6 +99,6 @@
       origin = "0.0642 0 0.0831"
       axis = "0 1 0"
-      min_deg = "-40"
-      max_deg = "70"
+      min_deg = "-10"
+      max_deg = "80"
       velocity = "58"
       effort = "20"
@@ -112,5 +112,5 @@
       origin = "0 0 0.3050"
       axis = "0 1 0"
-      min_deg = "-140"
+      min_deg = "-80"
       max_deg = "140"
       velocity = "158"
@@ -126,5 +126,5 @@
       axis = "0 0 1"
       min_deg = "-95"
-      max_deg = "158"
+      max_deg = "100"
       velocity = "238"
       effort = "3"
@@ -139,5 +139,5 @@
       axis = "0 1 0"
       min_deg = "-84"
-      max_deg = "105"
+      max_deg = "98"
       velocity = "198"
       effort = "0.1"
@@ -158,5 +158,5 @@
     <!-- Fixed joint between gripper and last link -->
     <joint name="${prefix}_gripper_base_joint" type="fixed">
-      <origin xyz="0 0 0.016" rpy="0 0 0" />
+      <origin xyz="0 0 0.016" rpy="0 0 ${-pi / 6}" />
       <parent link="${prefix}_link_5" />
       <child link="${prefix}_link_gripper" />
@@ -164,5 +164,5 @@
     <!-- Fixed joint between gripper and TOF optical frame -->
     <joint name="${prefix}_tof_optical_joint" type="fixed">
-      <origin xyz="0 0 0.09" rpy="0 0 ${pi / 2}" />
+      <origin xyz="0 0 0.09" rpy="0 0 0" />
       <parent link="${prefix}_link_gripper" />
       <child link="tof_optical_frame_id" />
@@ -170,5 +170,5 @@
     <!-- Fixed joint between link 4 and eef_aruco -->
     <joint name="${prefix}_eef_aruco_joint" type="fixed">
-      <origin xyz="0 0 -0.06" rpy="0 ${pi} 0" />
+      <origin xyz="0 0 -0.06" rpy="0 ${pi} ${-pi / 2}" />
       <parent link="${prefix}_link_4_bias" />
       <child link="${prefix}_eef_aruco" />
