Commit message: Use correct assets

File: urdf/inc/create_link.xacro (robot description, xacro)
@@ -22,5 +22,5 @@
         <origin xyz="0 0 0" rpy="0 0 0"/>
         <geometry>
-          <mesh filename="package://${mesh_package}/meshes/visual/${mesh_name}.dae"/>
+          <mesh filename="package://${mesh_package}/meshes/visual/${mesh_name}.stl"/>
         </geometry>
       </visual>
@@ -28,5 +28,5 @@
         <origin xyz="0 0 0" rpy="0 0 0"/>
         <geometry>
-          <mesh filename="package://${mesh_package}/meshes/collision/${mesh_name}.stl"/>
+          <mesh filename="package://${mesh_package}/meshes/visual/${mesh_name}.stl"/>
         </geometry>
       </collision>

Commit message: Refactor for 2 cobots

File: urdf/inc/create_link.xacro (robot description, xacro)
@@ -6,16 +6,8 @@
 <robot xmlns:xacro="http://wiki.ros.org/xacro">
   <xacro:macro name="create_link" params="
-        link_name
-        mesh_package
-        mesh_name
-        inertial_xyz
-        inertial_rpy
-        mass
-        ixx
-        ixy
-        ixz
-        iyy
-        iyz
-        izz">
+    link_name
+    mesh_package
+    mesh_name
+  ">
     <link name="${link_name}">
       <visual>
@@ -31,9 +23,4 @@
         </geometry>
       </collision>
-      <inertial>
-        <origin xyz="${inertial_xyz}" rpy="${inertial_rpy}"/>
-        <mass value="${mass}"/>
-        <inertia ixx="${ixx}" ixy="${ixy}" ixz="${ixz}" iyy="${iyy}" iyz="${iyz}" izz="${izz}"/>
-      </inertial>
     </link>
   </xacro:macro>
