Commit message: Add static gripper to URDF

File: urdf/inc/create_ar3.xacro (robot description, xacro)
@@ -53,4 +53,12 @@
       mesh_name = "link_5"
     />
+    <!-- Gripper links -->
+    <xacro:create_link
+      link_name = "${prefix}_link_gripper"
+      mesh_package = "ar3_description"
+      mesh_name = "gripper"
+    />
+    <!-- Phantom link for gripper gearbox -->
+    <link name="${prefix}_link_gripper_phantom" />
     <!-- Fixed joint between AR3 base and parent link -->
     <joint name="${prefix}_base_joint" type="fixed">
@@ -126,4 +134,22 @@
       effort = "3"
     />
+    <!-- Fixed joint between gripper and last link -->
+    <joint name="${prefix}_gripper_base_joint" type="fixed">
+      <origin xyz="0 0 0.016" rpy="0 0 0" />
+      <parent link="${prefix}_link_5" />
+      <child link="${prefix}_link_gripper" />
+    </joint>
+    <!-- Gripper motor joint -->
+    <xacro:create_joint
+      name = "${prefix}_gripper"
+      parent = "${prefix}_link_gripper"
+      child = "${prefix}_link_gripper_phantom"
+      origin = "0 0 0"
+      axis = "0 0 1"
+      min_deg = "0"
+      max_deg = "180"
+      velocity = "0.5"
+      effort = "0.5"
+    />
   </xacro:macro>
 </robot>

Commit message: Add aruco eef

File: urdf/inc/create_ar3.xacro (robot description, xacro)
@@ -61,4 +61,6 @@
     <!-- Phantom link for gripper gearbox -->
     <link name="${prefix}_link_gripper_phantom" />
+    <!-- Aruco link -->
+    <link name="${prefix}_eef_aruco" />
     <!-- Fixed joint between AR3 base and parent link -->
     <joint name="${prefix}_base_joint" type="fixed">
@@ -140,4 +142,10 @@
       <child link="${prefix}_link_gripper" />
     </joint>
+    <!-- Fixed joint between link 4 and eef_aruco -->
+    <joint name="${prefix}_eef_aruco_joint" type="fixed">
+      <origin xyz="0 0 -0.06" rpy="0 ${pi} 0" />
+      <parent link="${prefix}_link_4" />
+      <child link="${prefix}_eef_aruco" />
+    </joint>
     <!-- Gripper motor joint -->
     <xacro:create_joint

Commit message: Add bias joints

File: urdf/inc/create_ar3.xacro (robot description, xacro)
@@ -53,4 +53,11 @@
       mesh_name = "link_5"
     />
+    <!-- Arm bias links -->
+    <link name="${prefix}_link_0_bias" />
+    <link name="${prefix}_link_1_bias" />
+    <link name="${prefix}_link_2_bias" />
+    <link name="${prefix}_link_3_bias" />
+    <link name="${prefix}_link_4_bias" />
+    <!-- <link name="${prefix}_link_5_bias" /> -->
     <!-- Gripper links -->
     <xacro:create_link
@@ -74,4 +81,6 @@
       parent = "${prefix}_base"
       child = "${prefix}_link_0"
+      bias_parent = "${prefix}_base"
+      bias_child = "${prefix}_link_0_bias"
       origin = "0 0 0.0872"
       axis = "0 0 1"
@@ -85,4 +94,6 @@
       parent = "${prefix}_link_0"
       child = "${prefix}_link_1"
+      bias_parent = "${prefix}_link_0_bias"
+      bias_child = "${prefix}_link_1_bias"
       origin = "0.0642 0 0.0831"
       axis = "0 1 0"
@@ -96,4 +107,6 @@
       parent = "${prefix}_link_1"
       child = "${prefix}_link_2"
+      bias_parent = "${prefix}_link_1_bias"
+      bias_child = "${prefix}_link_2_bias"
       origin = "0 0 0.3050"
       axis = "0 1 0"
@@ -107,4 +120,6 @@
       parent = "${prefix}_link_2"
       child = "${prefix}_link_3"
+      bias_parent = "${prefix}_link_2_bias"
+      bias_child = "${prefix}_link_3_bias"
       origin = "0 0 0.0356"
       axis = "0 0 1"
@@ -118,4 +133,6 @@
       parent = "${prefix}_link_3"
       child = "${prefix}_link_4"
+      bias_parent = "${prefix}_link_3_bias"
+      bias_child = "${prefix}_link_4_bias"
       origin = "0 0 0.1873"
       axis = "0 1 0"
@@ -145,5 +162,5 @@
     <joint name="${prefix}_eef_aruco_joint" type="fixed">
       <origin xyz="0 0 -0.06" rpy="0 ${pi} 0" />
-      <parent link="${prefix}_link_4" />
+      <parent link="${prefix}_link_4_bias" />
       <child link="${prefix}_eef_aruco" />
     </joint>

File: urdf/inc/create_joint.xacro (robot description, xacro)
@@ -5,4 +5,6 @@
     parent
     child
+    bias_parent
+    bias_child
     origin
     axis
@@ -24,4 +26,18 @@
       />
     </joint>
+    <xacro:unless value="${bias_parent == '' || bias_child == ''}">
+      <joint name="${name}_bias" type="revolute">
+        <parent link="${bias_parent}" />
+        <child link="${bias_child}" />
+        <origin xyz="${origin}" rpy="0 0 0" />
+        <axis xyz="${axis}" />
+        <limit
+          effort="${effort}"
+          lower="${min_deg*pi/180}"
+          upper="${max_deg*pi/180}"
+          velocity="${velocity*pi/180}"
+        />
+      </joint>
+    </xacro:unless>
   </xacro:macro>
 </robot>

Commit message: bleh

File: urdf/inc/create_ar3.xacro (robot description, xacro)
@@ -59,5 +59,5 @@
     <link name="${prefix}_link_3_bias" />
     <link name="${prefix}_link_4_bias" />
-    <!-- <link name="${prefix}_link_5_bias" /> -->
+    <link name="${prefix}_link_5_bias" />
     <!-- Gripper links -->
     <xacro:create_link
@@ -124,6 +124,6 @@
       origin = "0 0 0.0356"
       axis = "0 0 1"
-      min_deg = "-158"
-      max_deg = "95"
+      min_deg = "-95"
+      max_deg = "158"
       velocity = "238"
       effort = "3"
@@ -146,4 +146,6 @@
       parent = "${prefix}_link_4"
       child = "${prefix}_link_5"
+      bias_parent = "${prefix}_link_4_bias"
+      bias_child = "${prefix}_link_5_bias"
       origin = "0 0 0.0199"
       axis = "0 0 1"
@@ -170,4 +172,6 @@
       parent = "${prefix}_link_gripper"
       child = "${prefix}_link_gripper_phantom"
+      bias_parent = "none"
+      bias_child = "none"
       origin = "0 0 0"
       axis = "0 0 1"

File: urdf/inc/create_joint.xacro (robot description, xacro)
@@ -26,5 +26,5 @@
       />
     </joint>
-    <xacro:unless value="${bias_parent == '' || bias_child == ''}">
+    <xacro:unless value="${bias_parent == 'none' or bias_child == 'none'}">
       <joint name="${name}_bias" type="revolute">
         <parent link="${bias_parent}" />

Commit message: Add TOF optical frame

File: urdf/inc/create_ar3.xacro (robot description, xacro)
@@ -66,4 +66,5 @@
       mesh_name = "gripper"
     />
+    <link name="tof_optical_frame_id" />
     <!-- Phantom link for gripper gearbox -->
     <link name="${prefix}_link_gripper_phantom" />
@@ -161,4 +162,10 @@
       <child link="${prefix}_link_gripper" />
     </joint>
+    <!-- Fixed joint between gripper and TOF optical frame -->
+    <joint name="${prefix}_tof_optical_joint" type="fixed">
+      <origin xyz="0 0 0.09" rpy="0 0 ${pi / 2}" />
+      <parent link="${prefix}_link_gripper" />
+      <child link="tof_optical_frame_id" />
+    </joint>
     <!-- Fixed joint between link 4 and eef_aruco -->
     <joint name="${prefix}_eef_aruco_joint" type="fixed">
